File: SwitchBoard/SwitchBoard.kicad_sch (KiCad schematic)
At the start: 8 parts, among them SW1 SW_SPDT, SW2 SW_SPDT

Commit message: Updated README.md, and started adding things in
Other:
- company: (none) -> Thomas Weinhardt
- title: (none) -> Switch Board
Changed lines of the file:
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@@
 	(generator_version "8.0")
 	(paper "A4")
+	(title_block
+		(title "Switch Board")
+		(date "2024-12-30")
+		(rev "1")
+		(company "Thomas Weinhardt")
+	)
 	(junction
 		(at 152.4 104.14)
